Commit message: Update readme and add spot leg foot frame

File: description/urdf/spot_leg.description.urdf.xacro (robot description, xacro)
@@ -112,3 +112,9 @@
     </inertial>
   </link>
+  <joint name="foot_transform" type="fixed">
+    <origin xyz="-0.015 0 -0.362" rpy="0 0.7854 0" />
+    <parent link="fl_lleg"/>
+    <child link="fl_foot" />
+  </joint>
+  <link name="fl_foot"/>
 </robot>
