Commit message: improve ur5 F/T sensor inertia

File: description/urdf/ur5.description.urdf.xacro (robot description, xacro)
@@ -225,10 +225,10 @@
     <inertial>
       <!-- mass value="0.118"/ -->
-      <mass value="0.018"/>
+      <mass value="0.0118"/>
       <origin rpy="0 1.57079632679 0" xyz="0.016 0.0 0.0"/>
       <inertia
-        ixx="8.00e-05" ixy="0.0" ixz="0.0"
-        iyy="8.00e-05" iyz="0.0"
-        izz="1.40e-04"/>
+        ixx="3.3984e-06" ixy="0.0" ixz="0.0"
+        iyy="2.5842e-06" iyz="0.0"
+        izz="2.5842e-06"/>
     </inertial>
   </link>
