Commit message: Adjust controller_manager rate, and improve spot collisions

File: description/urdf/spot.description.urdf.xacro (robot description, xacro)
@@ -23,5 +23,5 @@
     <collision>
       <geometry>
-        <mesh filename="package://ros2_descriptions/description/meshes/spot/collision/body.stl" />
+        <box size="0.85 0.25 0.18"/>
       </geometry>
     </collision>
@@ -82,6 +82,7 @@
     </visual>
     <collision>
-      <geometry>
-        <mesh filename="package://ros2_descriptions/description/meshes/spot/collision/fl_uleg.stl" />
+      <origin xyz="0.0 0 -0.16"/>
+      <geometry>
+        <cylinder radius="0.04" length="0.34"/>
       </geometry>
     </collision>
@@ -112,6 +113,7 @@
     </visual>
     <collision>
-      <geometry>
-        <mesh filename="package://ros2_descriptions/description/meshes/spot/collision/fl_lleg.stl" />
+      <origin xyz="0.0 0 -0.336"/>
+      <geometry>
+        <sphere radius="0.0355"/>
       </geometry>
     </collision>
@@ -178,6 +180,7 @@
     </visual>
     <collision>
-      <geometry>
-        <mesh filename="package://ros2_descriptions/description/meshes/spot/collision/fr_uleg.stl" />
+      <origin xyz="0.0 0 -0.16"/>
+      <geometry>
+        <cylinder radius="0.04" length="0.34"/>
       </geometry>
     </collision>
@@ -208,6 +211,7 @@
     </visual>
     <collision>
-      <geometry>
-        <mesh filename="package://ros2_descriptions/description/meshes/spot/collision/fr_lleg.stl" />
+      <origin xyz="0.0 0 -0.336"/>
+      <geometry>
+        <sphere radius="0.0355"/>
       </geometry>
     </collision>
@@ -274,6 +278,7 @@
     </visual>
     <collision>
-      <geometry>
-        <mesh filename="package://ros2_descriptions/description/meshes/spot/collision/hl_uleg.stl" />
+      <origin xyz="0.0 0 -0.16"/>
+      <geometry>
+        <cylinder radius="0.04" length="0.34"/>
       </geometry>
     </collision>
@@ -304,6 +309,7 @@
     </visual>
     <collision>
-      <geometry>
-        <mesh filename="package://ros2_descriptions/description/meshes/spot/collision/hl_lleg.stl" />
+      <origin xyz="0.0 0 -0.336"/>
+      <geometry>
+        <sphere radius="0.0355"/>
       </geometry>
     </collision>
@@ -370,6 +376,7 @@
     </visual>
     <collision>
-      <geometry>
-        <mesh filename="package://ros2_descriptions/description/meshes/spot/collision/hr_uleg.stl" />
+      <origin xyz="0.0 0 -0.16"/>
+      <geometry>
+        <cylinder radius="0.04" length="0.34"/>
       </geometry>
     </collision>
@@ -400,6 +407,7 @@
     </visual>
     <collision>
-      <geometry>
-        <mesh filename="package://ros2_descriptions/description/meshes/spot/collision/hr_lleg.stl" />
+      <origin xyz="0.0 0 -0.336"/>
+      <geometry>
+        <sphere radius="0.0355"/>
       </geometry>
     </collision>
