Commit message: adjust manipulator links CoM

File: description/urdf/bravo7.description.urdf.xacro (robot description, xacro)
@@ -15,5 +15,5 @@
     <inertial>
       <mass value="1.850"/>
-      <origin rpy="0 0 0" xyz="-0.015 -0.001 0.002"/>
+      <origin rpy="0 0 0" xyz="0 0 0.015"/>
       <inertia
         ixx="0.0025280" ixy="0.0" ixz="0.0"
@@ -103,5 +103,5 @@
     <inertial>
       <mass value="2.120"/>
-      <origin rpy="0 0 0" xyz="0.022 -0.004 -0.176"/>
+      <origin rpy="0 0 0" xyz="0.022 0.004 -0.176"/>
       <inertia
         ixx="0.035166" ixy="0.0" ixz="0.0"
@@ -145,5 +145,5 @@
     <inertial>
       <mass value="1.330"/>
-      <origin rpy="0 0 0" xyz="0.034 0.003 -0.046"/>
+      <origin rpy="0 0 0" xyz="0.034 -0.003 -0.046"/>
       <inertia
         ixx="0.001809" ixy="0.0" ixz="0.0"
@@ -176,5 +176,5 @@
     <inertial>
       <mass value="1.330"/>
-      <origin rpy="0 0 0" xyz="0.028 -0.012 0.145"/>
+      <origin rpy="0 0 0" xyz="-0.028 0.012 0.050"/>
       <inertia
         ixx="0.001983" ixy="0.0" ixz="0.0"

Commit message: merge 1013 link mesh and compress some meshes

File: description/urdf/bravo7.description.urdf.xacro (robot description, xacro)
@@ -64,40 +64,12 @@
     <visual>
       <geometry>
-        <mesh filename="package://ros2_descriptions/description/meshes/bravo7/1013 B.stl"/>
-      </geometry>
-      <origin rpy="0 0 3.14159265359" xyz="0 0 0"/>
-      <material name="bblack"/>
-    </visual>
-    <visual>
-      <geometry>
-        <mesh filename="package://ros2_descriptions/description/meshes/bravo7/1030.stl"/>
-      </geometry>
-      <origin xyz="0.046 0 -0.05334" rpy="3.14159265359 0 3.14159265359"/>
-      <material name="bblack"/>
-    </visual>
-    <visual>
-      <geometry>
-        <mesh filename="package://ros2_descriptions/description/meshes/bravo7/1026 A.stl"/>
-      </geometry>
-      <origin xyz="0.046 0 -0.23534" rpy="3.14159265359 0 3.14159265359"/>
-      <material name="bblack"/>
-    </visual>
-    <collision>
-      <geometry>
-        <mesh filename="package://ros2_descriptions/description/meshes/bravo7/1013 B.stl"/>
-      </geometry>
-      <origin rpy="0 0 3.14159265359" xyz="0 0 0"/>
-    </collision>
-    <collision>
-      <geometry>
-        <mesh filename="package://ros2_descriptions/description/meshes/bravo7/1030.stl"/>
-      </geometry>
-      <origin xyz="0.046 0 -0.05334" rpy="3.14159265359 0 3.14159265359"/>
-    </collision>
-    <collision>
-      <geometry>
-        <mesh filename="package://ros2_descriptions/description/meshes/bravo7/1026 A.stl"/>
-      </geometry>
-      <origin xyz="0.046 0 -0.23534" rpy="3.14159265359 0 3.14159265359"/>
+        <mesh filename="package://ros2_descriptions/description/meshes/bravo7/1013_merged.stl"/>
+      </geometry>
+      <material name="bblack"/>
+    </visual>
+    <collision>
+      <geometry>
+        <mesh filename="package://ros2_descriptions/description/meshes/bravo7/1013_merged.stl"/>
+      </geometry>
     </collision>
     <inertial>

Commit message: Simplified mesh 1026

File: description/urdf/bravo7.description.urdf.xacro (robot description, xacro)
@@ -4,11 +4,11 @@
     <visual>
       <geometry>
-        <mesh filename="package://ros2_descriptions/description/meshes/bravo7/1019 A.stl"/>
-      </geometry>
-      <material name="bblack"/>
-    </visual>
-    <collision>
-      <geometry>
-        <mesh filename="package://ros2_descriptions/description/meshes/bravo7/1019 A.stl"/>
+        <mesh filename="package://ros2_descriptions/description/meshes/bravo7/1019.stl"/>
+      </geometry>
+      <material name="bblack"/>
+    </visual>
+    <collision>
+      <geometry>
+        <mesh filename="package://ros2_descriptions/description/meshes/bravo7/1019.stl"/>
       </geometry>
     </collision>
@@ -93,25 +93,14 @@
     <visual>
       <geometry>
-        <mesh filename="package://ros2_descriptions/description/meshes/bravo7/1026 B.stl"/>
-      </geometry>
-      <material name="bblack"/>
-    </visual>
-    <visual>
-      <geometry>
-        <mesh filename="package://ros2_descriptions/description/meshes/bravo7/1026 C.stl"/>
-      </geometry>
-      <origin xyz="0.0408 0 -0.0956" rpy="3.14159265359 0 0"/>
-      <material name="bblack"/>
-    </visual>
-    <collision>
-      <geometry>
-        <mesh filename="package://ros2_descriptions/description/meshes/bravo7/1026 B.stl"/>
-      </geometry>
-    </collision>
-    <collision>
-      <geometry>
-        <mesh filename="package://ros2_descriptions/description/meshes/bravo7/1026 C.stl"/>
-      </geometry>
-      <origin xyz="0.0408 0 -0.0956" rpy="3.14159265359 0 0"/>
+        <mesh filename="package://ros2_descriptions/description/meshes/bravo7/1026.stl"/>
+      </geometry>
+      <origin xyz="-0.0052 0 0"/>
+      <material name="bblack"/>
+    </visual>
+    <collision>
+      <geometry>
+        <mesh filename="package://ros2_descriptions/description/meshes/bravo7/1026.stl"/>
+      </geometry>
+      <origin xyz="-0.0052 0 0"/>
     </collision>
     <inertial>

Commit message: Simplifed 1023

File: description/urdf/bravo7.description.urdf.xacro (robot description, xacro)
@@ -98,10 +98,4 @@
       <material name="bblack"/>
     </visual>
-    <collision>
-      <geometry>
-        <mesh filename="package://ros2_descriptions/description/meshes/bravo7/1026.stl"/>
-      </geometry>
-      <origin xyz="-0.0052 0 0"/>
-    </collision>
     <inertial>
       <mass value="1.330"/>
@@ -124,5 +118,5 @@
     <visual>
       <geometry>
-        <mesh filename="package://ros2_descriptions/description/meshes/bravo7/1023 A.stl"/>
+        <mesh filename="package://ros2_descriptions/description/meshes/bravo7/1023.stl"/>
       </geometry>
       <origin xyz="0 0 0.0054" rpy="0 0 3.14159265359"/>
@@ -131,5 +125,5 @@
     <collision>
       <geometry>
-        <mesh filename="package://ros2_descriptions/description/meshes/bravo7/1023 A.stl"/>
+        <mesh filename="package://ros2_descriptions/description/meshes/bravo7/1023.stl"/>
       </geometry>
       <origin xyz="0 0 0.0054" rpy="0 0 3.14159265359"/>
@@ -155,26 +149,9 @@
     <visual>
       <geometry>
-        <mesh filename="package://ros2_descriptions/description/meshes/bravo7/1023 B.stl"/>
-      </geometry>
-      <material name="bblack"/>
-    </visual>
-    <visual>
-      <geometry>
-        <mesh filename="package://ros2_descriptions/description/meshes/bravo7/1023 C.stl"/>
-      </geometry>
-      <origin xyz="0.0408 0 -0.0956" rpy="3.14159265359 0 3.14159265359"/>
-      <material name="bblack"/>
-    </visual>
-    <collision>
-      <geometry>
-        <mesh filename="package://ros2_descriptions/description/meshes/bravo7/1023 B.stl"/>
-      </geometry>
-    </collision>
-    <collision>
-      <geometry>
-        <mesh filename="package://ros2_descriptions/description/meshes/bravo7/1023 C.stl"/>
-      </geometry>
-      <origin xyz="0.0408 0 -0.0956" rpy="3.14159265359 0 3.14159265359"/>
-    </collision>
+        <mesh filename="package://ros2_descriptions/description/meshes/bravo7/1026.stl"/>
+      </geometry>
+      <origin xyz="-0.0052 0.001 0"/>
+      <material name="bblack"/>
+    </visual>
     <inertial>
       <mass value="0.970"/>
