Commit message: Add Spot quadruped. Simplify UR5 control xacro

File: description/ros2_control/ur5.ros2_control.xacro (robot description, xacro)
@@ -1,15 +1,10 @@
 <?xml version="1.0"?>
 <robot xmlns:xacro="http://www.ros.org/wiki/xacro">
-  <xacro:macro name="ur5_control" params="use_gazebo:=^|true">
+  <xacro:macro name="ur5_control">
     <xacro:property name="robot_yaml" value="$(find ros2_descriptions)/config/ur5.yaml"/>
     <xacro:property name="config" value="${xacro.load_yaml(robot_yaml)}"/>
     <ros2_control name="UR5RobotSystem" type="system">
       <hardware>
-        <xacro:if value="${use_gazebo}">
-          <plugin>gz_ros2_control/GazeboSimSystem</plugin>
-        </xacro:if>
-        <xacro:unless value="${use_gazebo}">
-          <!-- Insert the robot hardware plugin here -->
-        </xacro:unless>
+        <plugin>gz_ros2_control/GazeboSimSystem</plugin>
       </hardware>
       <joint name="shoulder_pan_joint">

Commit message: Simplify UR5 URDF. Allow the description file to be parsed solely by Pinocchio in the controller

File: description/ros2_control/ur5.ros2_control.xacro (robot description, xacro)
@@ -4,4 +4,22 @@
     <xacro:property name="robot_yaml" value="$(find ros2_descriptions)/config/ur5.yaml"/>
     <xacro:property name="config" value="${xacro.load_yaml(robot_yaml)}"/>
+    <gazebo>
+      <plugin filename="gz_ros2_control-system" name="gz_ros2_control::GazeboSimROS2ControlPlugin">
+        <parameters>$(find ros2_descriptions)/config/controllers.yaml</parameters>
+      </plugin>
+    </gazebo>
+    <gazebo reference="ee_fixed_joint">
+      <provideFeedback>true</provideFeedback>
+      <preserveFixedJoint>true</preserveFixedJoint>
+      <sensor name="force_torque_sensor" type="force_torque">
+        <update_rate>100</update_rate>
+        <always_on>true</always_on>
+        <topic>end_effector_ft_sensor</topic>
+        <force_torque>
+          <frame>sensor</frame>
+          <measure_direction>child_to_parent</measure_direction>
+        </force_torque>
+      </sensor>
+    </gazebo>
     <ros2_control name="UR5RobotSystem" type="system">
       <hardware>

File: description/ur5.urdf.xacro (robot description, xacro)
@@ -1,15 +1,12 @@
 <?xml version="1.0"?>
 <robot xmlns:xacro="http://www.ros.org/wiki/xacro" name="ur5">
-  <xacro:arg name="use_gazebo" default="false" />
+  <link name="world"/>
+  <joint name="support_joint" type="fixed">
+    <origin xyz="0 0 0.2" rpy="0 0 0" />
+    <parent link="world"/>
+    <child link="base_link" />
+  </joint>
   <xacro:include filename="$(find ros2_descriptions)/description/urdf/ur5.description.urdf.xacro" />
   <xacro:include filename="$(find ros2_descriptions)/description/ros2_control/ur5.ros2_control.xacro" />
-  <link name="world"/>
-  <xacro:ur5_robot parent="world">
-    <origin xyz="0 0 0" rpy="0 0 0" />
-  </xacro:ur5_robot>
   <xacro:ur5_control/>
-  <xacro:if value="$(arg use_gazebo)">
-    <xacro:include filename="$(find ros2_descriptions)/description/gazebo/ur5.gazebo.xacro" />
-    <xacro:ur5_gazebo/>
-  </xacro:if>
 </robot>

File: description/urdf/ur5.description.urdf.xacro (robot description, xacro)
@@ -1,13 +1,7 @@
 <?xml version="1.0" encoding="utf-8"?>
 <robot xmlns:xacro="http://wiki.ros.org/xacro" name="ur5">
-  <xacro:macro name="ur5_robot" params="parent *origin">
   <material name="grey">
     <color rgba="0.2 0.2 0.2 1.0"/>
   </material>
-  <joint name="base_joint" type="fixed">
-    <parent link="${parent}"/>
-    <child link="base_link" />
-    <xacro:insert_block name="origin" />
-  </joint>
   <link name="base_link">
     <visual>
@@ -239,4 +233,3 @@
     </inertial>
   </link>
-  </xacro:macro>
 </robot>

Commit message: Feat spot, and spot_leg models (#2)
* Add Spot quadruped. Simplify UR5 control xacro

* Add Spot single leg URDF, and refact it to be parsed standalone by the controller

* Simplify UR5 URDF. Allow the description file to be standalone by the controller

File: description/ros2_control/ur5.ros2_control.xacro (robot description, xacro)
@@ -1,15 +1,28 @@
 <?xml version="1.0"?>
 <robot xmlns:xacro="http://www.ros.org/wiki/xacro">
-  <xacro:macro name="ur5_control" params="use_gazebo:=^|true">
+  <xacro:macro name="ur5_control">
     <xacro:property name="robot_yaml" value="$(find ros2_descriptions)/config/ur5.yaml"/>
     <xacro:property name="config" value="${xacro.load_yaml(robot_yaml)}"/>
+    <gazebo>
+      <plugin filename="gz_ros2_control-system" name="gz_ros2_control::GazeboSimROS2ControlPlugin">
+        <parameters>$(find ros2_descriptions)/config/controllers.yaml</parameters>
+      </plugin>
+    </gazebo>
+    <gazebo reference="ee_fixed_joint">
+      <provideFeedback>true</provideFeedback>
+      <preserveFixedJoint>true</preserveFixedJoint>
+      <sensor name="force_torque_sensor" type="force_torque">
+        <update_rate>100</update_rate>
+        <always_on>true</always_on>
+        <topic>end_effector_ft_sensor</topic>
+        <force_torque>
+          <frame>sensor</frame>
+          <measure_direction>child_to_parent</measure_direction>
+        </force_torque>
+      </sensor>
+    </gazebo>
     <ros2_control name="UR5RobotSystem" type="system">
       <hardware>
-        <xacro:if value="${use_gazebo}">
-          <plugin>gz_ros2_control/GazeboSimSystem</plugin>
-        </xacro:if>
-        <xacro:unless value="${use_gazebo}">
-          <!-- Insert the robot hardware plugin here -->
-        </xacro:unless>
+        <plugin>gz_ros2_control/GazeboSimSystem</plugin>
       </hardware>
       <joint name="shoulder_pan_joint">

File: description/urdf/ur5.description.urdf.xacro (robot description, xacro)
@@ -1,13 +1,7 @@
 <?xml version="1.0" encoding="utf-8"?>
-<robot xmlns:xacro="http://wiki.ros.org/xacro">
-  <xacro:macro name="ur5_robot" params="parent *origin">
+<robot xmlns:xacro="http://wiki.ros.org/xacro" name="ur5">
   <material name="grey">
     <color rgba="0.2 0.2 0.2 1.0"/>
   </material>
-  <joint name="base_joint" type="fixed">
-    <parent link="${parent}"/>
-    <child link="base_link" />
-    <xacro:insert_block name="origin" />
-  </joint>
   <link name="base_link">
     <visual>
@@ -239,4 +233,3 @@
     </inertial>
   </link>
-  </xacro:macro>
 </robot>
