Commit message: Update root link name and add IMU sensor

File: description/ros2_control/spot.ros2_control.xacro (robot description, xacro)
@@ -134,4 +134,67 @@
       </joint>
     </ros2_control>
+  <!-- IMU sensor -->
+  <gazebo reference="spot_root">
+    <sensor name="imu_sensor" type="imu">
+      <gz_frame_id>spot_root</gz_frame_id>
+      <topic>spot_trunk/imu</topic>
+      <update_rate>250</update_rate>
+      <always_on>1</always_on>
+      <imu>
+        <angular_velocity>
+          <x>
+            <noise type="gaussian">
+              <mean>0</mean>
+              <stddev>0.0003394</stddev>
+              <dynamic_bias_stddev>3.8785e-05</dynamic_bias_stddev>
+              <dynamic_bias_correlation_time>1000</dynamic_bias_correlation_time>
+            </noise>
+          </x>
+          <y>
+            <noise type="gaussian">
+              <mean>0</mean>
+              <stddev>0.0003394</stddev>
+              <dynamic_bias_stddev>3.8785e-05</dynamic_bias_stddev>
+              <dynamic_bias_correlation_time>1000</dynamic_bias_correlation_time>
+            </noise>
+          </y>
+          <z>
+            <noise type="gaussian">
+              <mean>0</mean>
+              <stddev>0.0003394</stddev>
+              <dynamic_bias_stddev>3.8785e-05</dynamic_bias_stddev>
+              <dynamic_bias_correlation_time>1000</dynamic_bias_correlation_time>
+            </noise>
+          </z>
+        </angular_velocity>
+        <linear_acceleration>
+          <x>
+            <noise type="gaussian">
+              <mean>0</mean>
+              <stddev>0.004</stddev>
+              <dynamic_bias_stddev>0.006</dynamic_bias_stddev>
+              <dynamic_bias_correlation_time>300</dynamic_bias_correlation_time>
+            </noise>
+          </x>
+          <y>
+            <noise type="gaussian">
+              <mean>0</mean>
+              <stddev>0.004</stddev>
+              <dynamic_bias_stddev>0.006</dynamic_bias_stddev>
+              <dynamic_bias_correlation_time>300</dynamic_bias_correlation_time>
+            </noise>
+          </y>
+          <z>
+            <noise type="gaussian">
+              <mean>0</mean>
+              <stddev>0.004</stddev>
+              <dynamic_bias_stddev>0.006</dynamic_bias_stddev>
+              <dynamic_bias_correlation_time>300</dynamic_bias_correlation_time>
+            </noise>
+          </z>
+        </linear_acceleration>
+      </imu>
+    </sensor>
+  </gazebo>
   </xacro:macro>
 </robot>

File: description/urdf/spot.description.urdf.xacro (robot description, xacro)
@@ -8,11 +8,11 @@
   </material>
   <!-- This link is to suppress KDL parsing warning. -->
-  <link name="body_dummy"/>
-  <joint name="trunk_dummy" type="fixed">
-    <origin xyz="0 0 0.4" rpy="0 0 0" />
-    <parent link="body_dummy"/>
-    <child link="body" />
-  </joint>
-  <link name="body">
+  <link name="spot_root"/>
+  <joint name="trunk_root" type="fixed">
+    <origin xyz="0 0 -0.01" rpy="0 0 0" />
+    <parent link="spot_root"/>
+    <child link="spot_trunk" />
+  </joint>
+  <link name="spot_trunk">
     <visual>
       <geometry>
@@ -22,6 +22,7 @@
     </visual>
     <collision>
-      <geometry>
-        <box size="0.85 0.25 0.18"/>
+      <origin rpy="0 1.57079632679 0"/>
+      <geometry>
+        <cylinder radius="0.120" length="0.85"/>
       </geometry>
     </collision>
@@ -40,5 +41,5 @@
     <origin xyz="0.29785 0.05500 0.00000" rpy="0 0 0"/>
     <axis xyz="1 0 0"/>
-    <parent link="body"/>
+    <parent link="spot_trunk"/>
     <child link="fl_hip"/>
     <limit effort="999.9" velocity="999.9" lower="-0.7853981634" upper="0.7853981634"/>
@@ -138,5 +139,5 @@
     <origin xyz="0.29785 -0.05500 0.00000" rpy="0 0 0"/>
     <axis xyz="1 0 0"/>
-    <parent link="body"/>
+    <parent link="spot_trunk"/>
     <child link="fr_hip"/>
     <limit effort="999.9" velocity="999.9" lower="-0.78539816339744827899" upper="0.78539816339744827899"/>
@@ -236,5 +237,5 @@
     <origin xyz="-0.29785 0.05500 0.00000" rpy="0 0 0"/>
     <axis xyz="1 0 0"/>
-    <parent link="body"/>
+    <parent link="spot_trunk"/>
     <child link="hl_hip"/>
     <limit effort="999.9" velocity="999.9" lower="-0.78539816339744827899" upper="0.78539816339744827899"/>
@@ -334,5 +335,5 @@
     <origin xyz="-0.29785 -0.05500 0.00000" rpy="0 0 0"/>
     <axis xyz="1 0 0"/>
-    <parent link="body"/>
+    <parent link="spot_trunk"/>
     <child link="hr_hip"/>
     <limit effort="999.9" velocity="999.9" lower="-0.78539816339744827899" upper="0.78539816339744827899"/>
