Commit message: Refact spot_leg to be parsed standalone by the controller

File: description/ros2_control/spot_leg.ros2_control.xacro (robot description, xacro)
@@ -13,4 +13,11 @@
         <plugin>gz_ros2_control/GazeboSimSystem</plugin>
       </hardware>
+      <joint name="support_joint">
+        <state_interface name="position">
+          <param name="initial_value">0.0</param>
+        </state_interface>
+        <state_interface name="velocity"/>
+        <state_interface name="effort"/>
+      </joint>
       <joint name="fl_hipx">
         <command_interface name="effort"/>

File: description/spot_leg.urdf.xacro (robot description, xacro)
@@ -1,10 +1,15 @@
 <?xml version="1.0" ?>
 <robot xmlns:xacro="http://www.ros.org/wiki/xacro" name="spot_leg">
+  <link name="world"/>
+  <joint name="support_joint" type="prismatic">
+    <origin xyz="0 0 0.4" rpy="0 0 0" />
+    <axis xyz="0 0 1"/>
+    <parent link="world"/>
+    <child link="body"/>
+    <limit effort="999.9" velocity="340.0" lower="-0.15" upper="0.60"/>
+    <dynamics damping="0.08" friction="0.023"/>
+  </joint>
   <xacro:include filename="$(find ros2_descriptions)/description/urdf/spot_leg.description.urdf.xacro" />
   <xacro:include filename="$(find ros2_descriptions)/description/ros2_control/spot_leg.ros2_control.xacro" />
-  <link name="world"/>
-  <xacro:spot_robot parent="world">
-    <origin xyz="0 0 0.4" rpy="0 0 0" />
-  </xacro:spot_robot>
   <xacro:spot_control/>
 </robot>

File: description/urdf/spot_leg.description.urdf.xacro (robot description, xacro)
@@ -1,5 +1,4 @@
 <?xml version="1.0" encoding="utf-8"?>
-<robot xmlns:xacro="http://www.ros.org/wiki/xacro">
-  <xacro:macro name="spot_robot" params="parent *origin">
+<robot xmlns:xacro="http://www.ros.org/wiki/xacro" name="spot_leg">
   <material name="yellow">
     <color rgba="1.0 0.8431 0.0 1.0"/>
@@ -8,12 +7,4 @@
     <color rgba="0.2 0.2 0.2 1.0"/>
   </material>
-  <joint name="support_joint" type="prismatic">
-    <xacro:insert_block name="origin" />
-    <axis xyz="0 0 1"/>
-    <parent link="${parent}"/>
-    <child link="body"/>
-    <limit effort="999.9" velocity="340.0" lower="-0.15" upper="0.60"/>
-    <dynamics damping="0.08" friction="0.023"/>
-  </joint>
   <link name="body">
     <inertial>
@@ -121,4 +112,3 @@
     </inertial>
   </link>
-  </xacro:macro>
 </robot>

File: description/urdf/ur5.description.urdf.xacro (robot description, xacro)
@@ -1,4 +1,4 @@
 <?xml version="1.0" encoding="utf-8"?>
-<robot xmlns:xacro="http://wiki.ros.org/xacro">
+<robot xmlns:xacro="http://wiki.ros.org/xacro" name="ur5">
   <xacro:macro name="ur5_robot" params="parent *origin">
   <material name="grey">

Commit message: Fix ros2_control for fixed joint by adding an argument

File: description/ros2_control/spot_leg.ros2_control.xacro (robot description, xacro)
@@ -1,5 +1,5 @@
 <?xml version="1.0"?>
 <robot xmlns:xacro="http://www.ros.org/wiki/xacro">
-  <xacro:macro name="spot_control">
+  <xacro:macro name="spot_control" params="fixed_support">
     <xacro:property name="robot_yaml" value="$(find ros2_descriptions)/config/spot.yaml"/>
     <xacro:property name="config" value="${xacro.load_yaml(robot_yaml)}"/>
@@ -13,11 +13,13 @@
         <plugin>gz_ros2_control/GazeboSimSystem</plugin>
       </hardware>
-      <joint name="support_joint">
-        <state_interface name="position">
-          <param name="initial_value">0.0</param>
-        </state_interface>
-        <state_interface name="velocity"/>
-        <state_interface name="effort"/>
-      </joint>
+      <xacro:unless value="${fixed_support}">
+        <joint name="support_joint">
+          <state_interface name="position">
+            <param name="initial_value">0.0</param>
+          </state_interface>
+          <state_interface name="velocity"/>
+          <state_interface name="effort"/>
+        </joint>
+      </xacro:unless>
       <joint name="fl_hipx">
         <command_interface name="effort"/>

File: description/spot_leg.urdf.xacro (robot description, xacro)
@@ -1,5 +1,5 @@
 <?xml version="1.0" ?>
 <robot xmlns:xacro="http://www.ros.org/wiki/xacro" name="spot_leg">
-  <xacro:arg name="fixed" default="false"/>
+  <xacro:arg name="fixed" default="true"/>
   <link name="world"/>
   <xacro:if value="$(arg fixed)">
@@ -22,4 +22,4 @@
   <xacro:include filename="$(find ros2_descriptions)/description/urdf/spot_leg.description.urdf.xacro" />
   <xacro:include filename="$(find ros2_descriptions)/description/ros2_control/spot_leg.ros2_control.xacro" />
-  <xacro:spot_control/>
+  <xacro:spot_control fixed_support="$(arg fixed)"/>
 </robot>

Commit message: Add pivot joint interfaces

File: description/ros2_control/spot_leg.ros2_control.xacro (robot description, xacro)
@@ -1,5 +1,5 @@
 <?xml version="1.0"?>
 <robot xmlns:xacro="http://www.ros.org/wiki/xacro">
-  <xacro:macro name="spot_control" params="fixed_support">
+  <xacro:macro name="spot_control" params="fixed_support walker_setup">
     <xacro:property name="robot_yaml" value="$(find ros2_descriptions)/config/spot.yaml"/>
     <xacro:property name="config" value="${xacro.load_yaml(robot_yaml)}"/>
@@ -22,4 +22,13 @@
         </joint>
       </xacro:unless>
+      <xacro:if value="${walker_setup}">
+        <joint name="pivot_joint">
+          <state_interface name="position">
+            <param name="initial_value">0.0</param>
+          </state_interface>
+          <state_interface name="velocity"/>
+          <state_interface name="effort"/>
+        </joint>
+      </xacro:if>
       <joint name="fl_hipx">
         <command_interface name="effort"/>

File: description/spot_leg.urdf.xacro (robot description, xacro)
@@ -95,4 +95,4 @@
   <xacro:include filename="$(find ros2_descriptions)/description/urdf/spot_leg.description.urdf.xacro" />
   <xacro:include filename="$(find ros2_descriptions)/description/ros2_control/spot_leg.ros2_control.xacro" />
-  <xacro:spot_control fixed_support="${bench_setup == 'fixed'}"/>
+  <xacro:spot_control fixed_support="${bench_setup == 'fixed'}" walker_setup="${bench_setup == 'walker'}"/>
 </robot>
