Commit message: Resolve trunk DoF and add feet frames

File: description/spot.urdf.xacro (robot description, xacro)
@@ -1,10 +1,8 @@
 <?xml version="1.0" ?>
 <robot xmlns:xacro="http://www.ros.org/wiki/xacro" name="spot">
+  <!-- With Gazebo Harmonic (v8.10), we suppress the world link and joint
+       in order to allow the robot trunk 6 DoF. -->
   <xacro:include filename="$(find ros2_descriptions)/description/urdf/spot.description.urdf.xacro" />
   <xacro:include filename="$(find ros2_descriptions)/description/ros2_control/spot.ros2_control.xacro" />
-  <link name="world"/>
-  <xacro:spot_robot parent="world">
-    <origin xyz="0 0 0.4" rpy="0 0 0" />
-  </xacro:spot_robot>
   <xacro:spot_control/>
 </robot>

File: description/urdf/spot.description.urdf.xacro (robot description, xacro)
@@ -1,15 +1,16 @@
 <?xml version="1.0" encoding="utf-8"?>
-<robot xmlns:xacro="http://www.ros.org/wiki/xacro">
-  <xacro:macro name="spot_robot" params="parent *origin">
+<robot xmlns:xacro="http://www.ros.org/wiki/xacro" name="spot">
   <material name="yellow">
-    <color rgba="1.0 0.8431 0.0 1.0"/>
+    <color rgba="1.0 0.894 0.0 1.0"/>
   </material>
   <material name="grey">
-    <color rgba="0.2 0.2 0.2 1.0"/>
+    <color rgba="0.337 0.349 0.380 1.0"/>
   </material>
-  <joint name="trunk_joint" type="fixed">
-    <parent link="${parent}"/>
+  <!-- This link is to suppress KDL parsing warning. -->
+  <link name="body_dummy"/>
+  <joint name="trunk_dummy" type="fixed">
+    <origin xyz="0 0 0.4" rpy="0 0 0" />
+    <parent link="body_dummy"/>
     <child link="body" />
-    <xacro:insert_block name="origin" />
   </joint>
   <link name="body">
@@ -126,4 +127,10 @@
     </inertial>
   </link>
+  <joint name="fl_foot_transform" type="fixed">
+    <origin xyz="-0.015 0 -0.362" rpy="0 0.7854 0" />
+    <parent link="fl_lleg"/>
+    <child link="fl_foot" />
+  </joint>
+  <link name="fl_foot"/>
   <joint name="fr_hipx" type="revolute">
     <origin xyz="0.29785 -0.05500 0.00000" rpy="0 0 0"/>
@@ -216,4 +223,10 @@
     </inertial>
   </link>
+  <joint name="fr_foot_transform" type="fixed">
+    <origin xyz="-0.015 0 -0.362" rpy="0 0.7854 0" />
+    <parent link="fr_lleg"/>
+    <child link="fr_foot" />
+  </joint>
+  <link name="fr_foot"/>
   <joint name="hl_hipx" type="revolute">
     <origin xyz="-0.29785 0.05500 0.00000" rpy="0 0 0"/>
@@ -306,4 +319,10 @@
     </inertial>
   </link>
+  <joint name="hl_foot_transform" type="fixed">
+    <origin xyz="-0.015 0 -0.362" rpy="0 0.7854 0" />
+    <parent link="hl_lleg"/>
+    <child link="hl_foot" />
+  </joint>
+  <link name="hl_foot"/>
   <joint name="hr_hipx" type="revolute">
     <origin xyz="-0.29785 -0.05500 0.00000" rpy="0 0 0"/>
@@ -396,4 +415,9 @@
     </inertial>
   </link>
-  </xacro:macro>
+  <joint name="hr_foot_transform" type="fixed">
+    <origin xyz="-0.015 0 -0.362" rpy="0 0.7854 0" />
+    <parent link="hr_lleg"/>
+    <child link="hr_foot" />
+  </joint>
+  <link name="hr_foot"/>
 </robot>

Commit message: Add floating base Spot and Bravo 7 (#6)
* Resolve Spot trunk DoFs and add feet frames

* Add Spot PosePublisher

* add Bravo 7 (optimized) model

File: description/spot.urdf.xacro (robot description, xacro)
@@ -1,10 +1,21 @@
 <?xml version="1.0" ?>
 <robot xmlns:xacro="http://www.ros.org/wiki/xacro" name="spot">
+  <!--
+    The 'world' link must be suppressed and the robot trunk is the root
+    link with all the free body 6-DoF. Through the PosePublisher plugin,
+    one can publish the model pose and visualize it properly on Rviz2.
+  -->
+  <gazebo>
+    <plugin
+      filename="gz-sim-pose-publisher-system"
+      name="gz::sim::systems::PosePublisher">
+      <use_pose_vector_msg>true</use_pose_vector_msg>
+      <publish_model_pose>true</publish_model_pose>
+      <publish_link_pose>false</publish_link_pose>
+      <update_frequency>50</update_frequency>
+    </plugin>
+  </gazebo>
   <xacro:include filename="$(find ros2_descriptions)/description/urdf/spot.description.urdf.xacro" />
   <xacro:include filename="$(find ros2_descriptions)/description/ros2_control/spot.ros2_control.xacro" />
-  <link name="world"/>
-  <xacro:spot_robot parent="world">
-    <origin xyz="0 0 0.4" rpy="0 0 0" />
-  </xacro:spot_robot>
   <xacro:spot_control/>
 </robot>

File: description/urdf/spot.description.urdf.xacro (robot description, xacro)
@@ -1,15 +1,16 @@
 <?xml version="1.0" encoding="utf-8"?>
-<robot xmlns:xacro="http://www.ros.org/wiki/xacro">
-  <xacro:macro name="spot_robot" params="parent *origin">
+<robot xmlns:xacro="http://www.ros.org/wiki/xacro" name="spot">
   <material name="yellow">
-    <color rgba="1.0 0.8431 0.0 1.0"/>
+    <color rgba="1.0 0.894 0.0 1.0"/>
   </material>
   <material name="grey">
-    <color rgba="0.2 0.2 0.2 1.0"/>
+    <color rgba="0.337 0.349 0.380 1.0"/>
   </material>
-  <joint name="trunk_joint" type="fixed">
-    <parent link="${parent}"/>
+  <!-- This link is to suppress KDL parsing warning. -->
+  <link name="body_dummy"/>
+  <joint name="trunk_dummy" type="fixed">
+    <origin xyz="0 0 0.4" rpy="0 0 0" />
+    <parent link="body_dummy"/>
     <child link="body" />
-    <xacro:insert_block name="origin" />
   </joint>
   <link name="body">
@@ -22,5 +23,5 @@
     <collision>
       <geometry>
-        <mesh filename="package://ros2_descriptions/description/meshes/spot/collision/body.stl" />
+        <box size="0.85 0.25 0.18"/>
       </geometry>
     </collision>
@@ -81,6 +82,7 @@
     </visual>
     <collision>
-      <geometry>
-        <mesh filename="package://ros2_descriptions/description/meshes/spot/collision/fl_uleg.stl" />
+      <origin xyz="0.0 0 -0.16"/>
+      <geometry>
+        <cylinder radius="0.04" length="0.34"/>
       </geometry>
     </collision>
@@ -111,6 +113,7 @@
     </visual>
     <collision>
-      <geometry>
-        <mesh filename="package://ros2_descriptions/description/meshes/spot/collision/fl_lleg.stl" />
+      <origin xyz="0.0 0 -0.336"/>
+      <geometry>
+        <sphere radius="0.0355"/>
       </geometry>
     </collision>
@@ -126,4 +129,10 @@
     </inertial>
   </link>
+  <joint name="fl_foot_transform" type="fixed">
+    <origin xyz="-0.015 0 -0.362" rpy="0 0.7854 0" />
+    <parent link="fl_lleg"/>
+    <child link="fl_foot" />
+  </joint>
+  <link name="fl_foot"/>
   <joint name="fr_hipx" type="revolute">
     <origin xyz="0.29785 -0.05500 0.00000" rpy="0 0 0"/>
@@ -171,6 +180,7 @@
     </visual>
     <collision>
-      <geometry>
-        <mesh filename="package://ros2_descriptions/description/meshes/spot/collision/fr_uleg.stl" />
+      <origin xyz="0.0 0 -0.16"/>
+      <geometry>
+        <cylinder radius="0.04" length="0.34"/>
       </geometry>
     </collision>
@@ -201,6 +211,7 @@
     </visual>
     <collision>
-      <geometry>
-        <mesh filename="package://ros2_descriptions/description/meshes/spot/collision/fr_lleg.stl" />
+      <origin xyz="0.0 0 -0.336"/>
+      <geometry>
+        <sphere radius="0.0355"/>
       </geometry>
     </collision>
@@ -216,4 +227,10 @@
     </inertial>
   </link>
+  <joint name="fr_foot_transform" type="fixed">
+    <origin xyz="-0.015 0 -0.362" rpy="0 0.7854 0" />
+    <parent link="fr_lleg"/>
+    <child link="fr_foot" />
+  </joint>
+  <link name="fr_foot"/>
   <joint name="hl_hipx" type="revolute">
     <origin xyz="-0.29785 0.05500 0.00000" rpy="0 0 0"/>
@@ -261,6 +278,7 @@
     </visual>
     <collision>
-      <geometry>
-        <mesh filename="package://ros2_descriptions/description/meshes/spot/collision/hl_uleg.stl" />
+      <origin xyz="0.0 0 -0.16"/>
+      <geometry>
+        <cylinder radius="0.04" length="0.34"/>
       </geometry>
     </collision>
@@ -291,6 +309,7 @@
     </visual>
     <collision>
-      <geometry>
-        <mesh filename="package://ros2_descriptions/description/meshes/spot/collision/hl_lleg.stl" />
+      <origin xyz="0.0 0 -0.336"/>
+      <geometry>
+        <sphere radius="0.0355"/>
       </geometry>
     </collision>
@@ -306,4 +325,10 @@
     </inertial>
   </link>
+  <joint name="hl_foot_transform" type="fixed">
+    <origin xyz="-0.015 0 -0.362" rpy="0 0.7854 0" />
+    <parent link="hl_lleg"/>
+    <child link="hl_foot" />
+  </joint>
+  <link name="hl_foot"/>
   <joint name="hr_hipx" type="revolute">
     <origin xyz="-0.29785 -0.05500 0.00000" rpy="0 0 0"/>
@@ -351,6 +376,7 @@
     </visual>
     <collision>
-      <geometry>
-        <mesh filename="package://ros2_descriptions/description/meshes/spot/collision/hr_uleg.stl" />
+      <origin xyz="0.0 0 -0.16"/>
+      <geometry>
+        <cylinder radius="0.04" length="0.34"/>
       </geometry>
     </collision>
@@ -381,6 +407,7 @@
     </visual>
     <collision>
-      <geometry>
-        <mesh filename="package://ros2_descriptions/description/meshes/spot/collision/hr_lleg.stl" />
+      <origin xyz="0.0 0 -0.336"/>
+      <geometry>
+        <sphere radius="0.0355"/>
       </geometry>
     </collision>
@@ -396,4 +423,9 @@
     </inertial>
   </link>
-  </xacro:macro>
+  <joint name="hr_foot_transform" type="fixed">
+    <origin xyz="-0.015 0 -0.362" rpy="0 0.7854 0" />
+    <parent link="hr_lleg"/>
+    <child link="hr_foot" />
+  </joint>
+  <link name="hr_foot"/>
 </robot>
