Commit message: clean Bravo 7 tree

File: description/bravo7.urdf.xacro (robot description, xacro)
@@ -3,7 +3,7 @@
   <link name="world">
     <visual>
-      <origin rpy="0 0 0" xyz="0 0 0.15"/>
+      <origin rpy="0 0 0" xyz="0 0 0.30"/>
       <geometry>
-        <cylinder radius="0.075" length="0.30"/>
+        <cylinder radius="0.075" length="0.60"/>
       </geometry>
       <material name="StaticBlue">
@@ -12,12 +12,12 @@
     </visual>
     <collision name="support_body">
-      <origin rpy="0 0 0" xyz="0 0 0.15"/>
+      <origin rpy="0 0 0" xyz="0 0 0.30"/>
       <geometry>
-        <cylinder radius="0.075" length="0.30"/>
+        <cylinder radius="0.075" length="0.60"/>
       </geometry>
     </collision>
   </link>
   <joint name="support_joint" type="fixed">
-    <origin xyz="-0.045 0 0.30" rpy="0 0 0"/>
+    <origin xyz="-0.045 0 0.60" rpy="0 0 0"/>
     <parent link="world"/>
     <child link="base_link"/>

File: description/urdf/bravo7.description.urdf.xacro (robot description, xacro)
@@ -98,4 +98,11 @@
       <material name="bblack"/>
     </visual>
+    <visual>
+      <geometry>
+        <mesh filename="package://ros2_descriptions/description/meshes/bravo7/1026 A.stl"/>
+      </geometry>
+      <origin xyz="0.046 0 -0.23534" rpy="3.14159265359 0 3.14159265359"/>
+      <material name="bblack"/>
+    </visual>
     <collision>
       <geometry>
@@ -119,47 +126,8 @@
     </inertial>
   </link>
-  <joint name="1013_end_joint" type="fixed">
+  <joint name="e_joint" type="revolute">
     <parent link="1013_joint_link"/>
-    <child link="1013_end_link"/>
-    <origin xyz="0.046 0 -0.05334" rpy="3.14159265359 0 3.14159265359"/>
-  </joint>
-  <link name="1013_end_link"/>
-  <joint name="e_base_joint" type="fixed">
-    <parent link="1013_end_link"/>
-    <child link="1026_0_base_link"/>
-    <origin xyz="0 0 0.182" rpy="0 0 0"/>
-  </joint>
-  <link name="1026_0_base_link">
-    <visual>
-      <geometry>
-        <mesh filename="package://ros2_descriptions/description/meshes/bravo7/1026 A.stl"/>
-      </geometry>
-      <material name="bblack"/>
-    </visual>
-    <collision>
-      <geometry>
-        <cylinder radius="0.0408" length="0.059"/>
-      </geometry>
-      <origin xyz="0 00 0.0295" rpy="0 0 0"/>
-    </collision>
-    <collision>
-      <geometry>
-        <cylinder radius="0.0408" length="0.0599"/>
-      </geometry>
-      <origin xyz="0.0408 -0.01435 0.059" rpy="1.57079632679 0 0"/>
-    </collision>
-    <inertial>
-      <mass value="1.000"/>
-      <origin rpy="0 0 0" xyz="0.0 0.0 0.25"/>
-      <inertia
-        ixx="0.031216803515624995" ixy="0.0" ixz="0.0"
-        iyy="0.031216803515624995" iyz="0.0"
-        izz="0.004095"/>
-    </inertial>
-  </link>
-  <joint name="e_joint" type="revolute">
-    <parent link="1026_0_base_link"/>
     <child link="1026_0_joint_link"/>
-    <origin xyz="0.0408 0 0.059" rpy="0 0 0"/>
+    <origin xyz="0.0052 0 -0.29434" rpy="3.14159265359 0 3.14159265359"/>
     <axis xyz="0 -1 0"/>
     <limit effort="110.0" velocity="0.7854" lower="0.0" upper="3.2"/>
@@ -173,4 +141,11 @@
       <material name="bblack"/>
     </visual>
+    <visual>
+      <geometry>
+        <mesh filename="package://ros2_descriptions/description/meshes/bravo7/1026 C.stl"/>
+      </geometry>
+      <origin xyz="0.0408 0 -0.0956" rpy="3.14159265359 0 0"/>
+      <material name="bblack"/>
+    </visual>
     <collision>
       <geometry>
@@ -194,57 +169,12 @@
     </inertial>
   </link>
-  <joint name="1026_0_end_joint" type="fixed">
+  <joint name="d_joint" type="continuous">
     <parent link="1026_0_joint_link"/>
-    <child link="1026_0_end_link"/>
+    <child link="1023_0_base_link"/>
     <origin xyz="0.0408 0 -0.0956" rpy="3.14159265359 0 0"/>
-  </joint>
-  <link name="1026_0_end_link"/>
-  <joint name="d_base_joint" type="fixed">
-    <parent link="1026_0_end_link"/>
-    <child link="1026_1_base_link"/>
-    <origin xyz="0 0 0" rpy="0 0 0"/>
-  </joint>
-  <link name="1026_1_base_link"/>
-  <joint name="d_joint" type="continuous">
-    <parent link="1026_1_base_link"/>
-    <child link="1026_1_joint_link"/>
-    <origin xyz="0 0 0" rpy="0 0 0"/>
     <axis xyz="0 0 -1"/>
     <limit effort="110.0" velocity="0.7854"/>
     <dynamics damping="0.0" friction="0.07"/>
   </joint>
-  <link name="1026_1_joint_link">
-    <visual>
-      <geometry>
-        <mesh filename="package://ros2_descriptions/description/meshes/bravo7/1026 C.stl"/>
-      </geometry>
-      <material name="bblack"/>
-    </visual>
-    <collision>
-      <geometry>
-        <cylinder radius="0.0408" length="0.003"/>
-      </geometry>
-      <origin xyz="0 0 0" rpy="0 0 3.14159265359"/>
-    </collision>
-    <inertial>
-      <mass value="1.2190"/>
-      <origin rpy="0 0 0" xyz="0.0 0.0 0.0"/>
-      <inertia
-        ixx="0.002013889583333333" ixy="0.0" ixz="0.0"
-        iyy="0.002013889583333333" iyz="0.0"
-        izz="0.0021942"/>
-    </inertial>
-  </link>
-  <joint name="1026_1_end_joint" type="fixed">
-    <parent link="1026_1_joint_link"/>
-    <child link="1026_1_end_link"/>
-    <origin xyz="0 0 0.0054" rpy="0 0 3.14159265359"/>
-  </joint>
-  <link name="1026_1_end_link"/>
-  <joint name="c_base_joint" type="fixed">
-    <parent link="1026_1_end_link"/>
-    <child link="1023_0_base_link"/>
-    <origin xyz="0 0 0" rpy="0 0 0"/>
-  </joint>
   <link name="1023_0_base_link">
     <visual>
@@ -252,4 +182,5 @@
         <mesh filename="package://ros2_descriptions/description/meshes/bravo7/1023 A.stl"/>
       </geometry>
+      <origin xyz="0 0 0.0054" rpy="0 0 3.14159265359"/>
       <material name="bblack"/>
     </visual>
@@ -278,5 +209,5 @@
     <parent link="1023_0_base_link"/>
     <child link="1023_0_joint_link"/>
-    <origin xyz="0.0408 0 0.059" rpy="0 0 0"/>
+    <origin xyz="-0.0408 0 0.0644" rpy="0 0 3.14159265359"/>
     <axis xyz="0 -1 0"/>
     <limit effort="110.0" velocity="0.7854" lower="0.0" upper="3.2"/>
@@ -290,4 +221,11 @@
       <material name="bblack"/>
     </visual>
+    <visual>
+      <geometry>
+        <mesh filename="package://ros2_descriptions/description/meshes/bravo7/1023 C.stl"/>
+      </geometry>
+      <origin xyz="0.0408 0 -0.0956" rpy="3.14159265359 0 3.14159265359"/>
+      <material name="bblack"/>
+    </visual>
     <collision>
       <geometry>
@@ -311,34 +249,23 @@
     </inertial>
   </link>
-  <joint name="1023_0_end_joint" type="fixed">
+  <joint name="b_joint" type="continuous">
     <parent link="1023_0_joint_link"/>
-    <child link="1023_0_end_link"/>
-    <origin xyz="0.0408 0 -0.0956" rpy="3.14159265359 0 0"/>
-  </joint>
-  <link name="1023_0_end_link"/>
-  <joint name="b_base_joint" type="fixed">
-    <parent link="1023_0_end_link"/>
-    <child link="1023_1_base_link"/>
-    <origin xyz="0 0 0" rpy="0 0 0"/>
-  </joint>
-  <link name="1023_1_base_link"/>
-  <joint name="b_joint" type="continuous">
-    <parent link="1023_1_base_link"/>
-    <child link="1023_1_joint_link"/>
-    <origin xyz="0 0 0" rpy="0 0 3.14159265359"/>
+    <child link="1038_base_link"/>
+    <origin xyz="0.0408 0 -0.0956" rpy="3.14159265359 0 3.14159265359"/>
     <axis xyz="0 0 -1"/>
     <limit effort="110.0" velocity="0.7854"/>
     <dynamics damping="0.0" friction="0.07"/>
   </joint>
-  <link name="1023_1_joint_link">
-    <visual>
-      <geometry>
-        <mesh filename="package://ros2_descriptions/description/meshes/bravo7/1023 C.stl"/>
-      </geometry>
-      <material name="bblack"/>
-    </visual>
-    <collision>
-      <geometry>
-        <cylinder radius="0.0408" length="0.003"/>
+  <link name="1038_base_link">
+    <visual>
+      <geometry>
+        <mesh filename="package://ros2_descriptions/description/meshes/bravo7/1038.stl"/>
+      </geometry>
+      <origin xyz="0 0 0.0054" rpy="0 0 0"/>
+      <material name="bblack"/>
+    </visual>
+    <collision>
+      <geometry>
+        <cylinder radius="0.0408" length="0.12535"/>
       </geometry>
     </collision>
@@ -352,34 +279,8 @@
     </inertial>
   </link>
-  <joint name="1023_1_end_joint" type="fixed">
-    <parent link="1023_1_joint_link"/>
-    <child link="1038_base_link"/>
-    <origin xyz="0 0 0.0054" rpy="0 0 0"/>
-  </joint>
-  <link name="1038_base_link">
-    <visual>
-      <geometry>
-        <mesh filename="package://ros2_descriptions/description/meshes/bravo7/1038.stl"/>
-      </geometry>
-      <material name="bblack"/>
-    </visual>
-    <collision>
-      <geometry>
-        <cylinder radius="0.0408" length="0.12535"/>
-      </geometry>
-    </collision>
-    <inertial>
-      <mass value="0.18790"/>
-      <origin rpy="0 0 0" xyz="0.0 0.0 0.0"/>
-      <inertia
-        ixx="8.062475833333332e-05" ixy="0.0" ixz="0.0"
-        iyy="8.062475833333332e-05" iyz="0.0"
-        izz="0.0001321171875"/>
-    </inertial>
-  </link>
   <joint name="1038_end_joint" type="fixed">
     <parent link="1038_base_link"/>
     <child link="jaws_base_link"/>
-    <origin xyz="0 0 0.12535" rpy="0 -1.57079632679 0"/>
+    <origin xyz="0 0 0.13075" rpy="0 -1.57079632679 0"/>
   </joint>
   <link name="jaws_base_link"/>

Commit message: add half of the jaws, and start inertial params definition. CoM and Ixx must be adjusted

File: description/bravo7.urdf.xacro (robot description, xacro)
@@ -1,4 +1,7 @@
 <?xml version="1.0"?>
 <robot xmlns:xacro="http://www.ros.org/wiki/xacro" name="Bravo7">
+  <material name="bblack">
+    <color rgba="0.3 0.3 0.3 1"/>
+  </material>
   <link name="world">
     <visual>
@@ -19,9 +22,78 @@
   </link>
   <joint name="support_joint" type="fixed">
-    <origin xyz="-0.045 0 0.60" rpy="0 0 0"/>
     <parent link="world"/>
     <child link="base_link"/>
+    <origin xyz="-0.045 0 0.60" rpy="0 0 0"/>
   </joint>
+  <!-- manipulator without jaws, for Pinocchio lib -->
   <xacro:include filename="$(find ros2_descriptions)/description/urdf/bravo7.description.urdf.xacro"/>
+  <joint name="a_joint" type="prismatic">
+    <!-- this parent link is the last link in bravo7.description -->
+    <parent link="jaws_base_link"/>
+    <child link="jaws_push_rod_link"/>
+    <origin rpy="0 0 0" xyz="0.009 0 0"/>
+    <axis xyz="1 0 0"/>
+    <limit lower="0.000" upper="0.010" effort="10" velocity="10"/>
+    <dynamics damping="0.14833" friction="13.166"/>
+  </joint>
+  <!-- dummy frame for the prismatic joint -->
+  <link name="jaws_push_rod_link"/>
+  <joint name="jaws_base_joint" type="fixed">
+    <parent link="jaws_base_link"/>
+    <child link="jaws_handle_link"/>
+    <origin xyz="0 0 0" rpy="0 0 0"/>
+  </joint>
+  <link name="jaws_handle_link">
+    <visual>
+      <geometry>
+        <mesh filename="package://ros2_descriptions/description/meshes/bravo7/RS2-257.stl"/>
+      </geometry>
+      <material name="bblack"/>
+    </visual>
+    <collision>
+      <geometry>
+        <mesh filename="package://ros2_descriptions/description/meshes/bravo7/RS2-257.stl"/>
+      </geometry>
+    </collision>
+    <inertial>
+      <mass value="0.44"/>
+      <origin rpy="0 0 0" xyz="0.0 0.0 0.0"/>
+      <inertia
+        ixx="0.000309" ixy="0.0" ixz="0.0"
+        iyy="0.002237" iyz="0.0"
+        izz="0.002258"/>
+    </inertial>
+  </link>
+  <joint name="rs2_300_joint" type="revolute">
+    <parent link="jaws_handle_link"/>
+    <child link="rs2_300_link"/>
+    <origin xyz="0.0241 0.0268 0" rpy="0 0 0"/>
+    <axis xyz="0 0 1"/>
+    <limit lower="0" upper="1.0" effort="10" velocity="10"/>
+    <mimic joint="a_joint" multiplier="54" offset="0"/>
+  </joint>
+  <link name="rs2_300_link">
+    <visual>
+      <geometry>
+        <mesh filename="package://ros2_descriptions/description/meshes/bravo7/RS2-300.stl"/>
+      </geometry>
+      <origin rpy="3.14159265359 0 0" xyz="0.0 0.0 0.0"/>
+      <material name="bblack"/>
+    </visual>
+    <collision>
+      <geometry>
+        <mesh filename="package://ros2_descriptions/description/meshes/bravo7/RS2-300.stl"/>
+      </geometry>
+      <origin rpy="3.14159265359 0 0" xyz="0.0 0.0 0.0"/>
+    </collision>
+    <inertial>
+      <mass value="0.10"/>
+      <origin rpy="0 0 0" xyz="0.0 0.0 0.0"/>
+      <inertia
+        ixx="0.000050" ixy="0.0" ixz="0.0"
+        iyy="0.000372" iyz="0.0"
+        izz="0.000376"/>
+    </inertial>
+  </link>
   <xacro:include filename="$(find ros2_descriptions)/description/ros2_control/bravo7.ros2_control.xacro"/>
   <xacro:bravo7_control/>

File: description/urdf/bravo7.description.urdf.xacro (robot description, xacro)
@@ -1,7 +1,4 @@
 <?xml version="1.0" encoding="utf-8"?>
 <robot xmlns:xacro="http://wiki.ros.org/xacro" name="Bravo7">
-  <material name="bblack">
-    <color rgba="0.3 0.3 0.3 1"/>
-  </material>
   <link name="base_link">
     <visual>
@@ -13,27 +10,14 @@
     <collision>
       <geometry>
-        <box size="0.0625 0.1112 0.088"/>
-      </geometry>
-      <origin rpy="0 0 0" xyz="0.03625 0 0.044"/>
-    </collision>
-    <collision>
-      <geometry>
-        <box size="0.050 0.080 0.060"/>
-      </geometry>
-      <origin rpy="0 0 0" xyz="0.030 -0.04556 0.03"/>
-    </collision>
-    <collision>
-      <geometry>
-        <cylinder radius="0.046" length="0.0851"/>
-      </geometry>
-      <origin rpy="0 0 0" xyz="0.0675 0 0.04255"/>
-    </collision>
-    <inertial>
-      <mass value="1.2000"/>
-      <origin rpy="0 0 0" xyz="0.0 0.0 0.0"/>
-      <inertia
-        ixx="0.00443333156" ixy="0.0" ixz="0.0"
-        iyy="0.00443333156" iyz="0.0"
-        izz="0.0072"/>
+        <mesh filename="package://ros2_descriptions/description/meshes/bravo7/1019 A.stl"/>
+      </geometry>
+    </collision>
+    <inertial>
+      <mass value="1.850"/>
+      <origin rpy="0 0 0" xyz="-0.015 -0.001 0.002"/>
+      <inertia
+        ixx="0.0025280" ixy="0.0" ixz="0.0"
+        iyy="0.0025930" iyz="0.0"
+        izz="0.0033120"/>
     </inertial>
   </link>
@@ -44,5 +28,5 @@
     <axis xyz="0 0 -1"/>
     <limit effort="110.0" velocity="0.7854"/>
-    <dynamics damping="0.0" friction="0.09"/>
+    <dynamics damping="1430.0" friction="0.079"/>
   </joint>
   <link name="1013_base_link">
@@ -56,21 +40,15 @@
     <collision>
       <geometry>
-        <cylinder radius="0.046" length="0.0667"/>
-      </geometry>
-      <origin rpy="0 0 0" xyz="0.0 0.0 0.03335"/>
-    </collision>
-    <collision>
-      <geometry>
-        <cylinder radius="0.046" length="0.0738"/>
-      </geometry>
-      <origin rpy="1.57079632679 0 0 " xyz="0.046 0.0149 0.0667"/>
-    </collision>
-    <inertial>
-      <mass value="2.3930"/>
-      <origin rpy="0 0 0" xyz="0.0 0.0 0.28"/>
-      <inertia
-        ixx="0.13388583541666665" ixy="0.0" ixz="0.0"
-        iyy="0.13388583541666665" iyz="0.0"
-        izz="0.0151074"/>
+        <mesh filename="package://ros2_descriptions/description/meshes/bravo7/1013 A.stl"/>
+      </geometry>
+      <origin rpy="0 0 3.14159265359" xyz="0 0 0"/>
+    </collision>
+    <inertial>
+      <mass value="1.620"/>
+      <origin rpy="0 0 0" xyz="0.031 -0.010 0.098"/>
+      <inertia
+        ixx="0.003180" ixy="0.0" ixz="0.0"
+        iyy="0.004209" iyz="0.0"
+        izz="0.002387"/>
     </inertial>
   </link>
@@ -81,5 +59,5 @@
     <axis xyz="0 -1 0"/>
     <limit effort="110.0" velocity="0.7854" lower="0.0" upper="3.2"/>
-    <dynamics damping="0.0" friction="0.09"/>
+    <dynamics damping="1430.0" friction="0.079"/>
   </joint>
   <link name="1013_joint_link">
@@ -107,21 +85,27 @@
     <collision>
       <geometry>
-        <cylinder radius="0.046" length="0.0228"/>
-      </geometry>
-      <origin rpy="1.57079632679 0 0 " xyz="0 -0.0334 0"/>
-    </collision>
-    <collision>
-      <geometry>
-        <cylinder radius="0.046" length="0.05094"/>
-      </geometry>
-      <origin rpy="0 0 0" xyz="0.046 0 -0.02547"/>
-    </collision>
-    <inertial>
-      <mass value="4.00"/>
-      <origin rpy="0 0 0" xyz="0.0 0.0 0.25"/>
-      <inertia
-        ixx="0.0603515624995" ixy="0.0" ixz="0.0"
-        iyy="0.0603515624995" iyz="0.0"
-        izz="0.0076"/>
+        <mesh filename="package://ros2_descriptions/description/meshes/bravo7/1013 B.stl"/>
+      </geometry>
+      <origin rpy="0 0 3.14159265359" xyz="0 0 0"/>
+    </collision>
+    <collision>
+      <geometry>
+        <mesh filename="package://ros2_descriptions/description/meshes/bravo7/1030.stl"/>
+      </geometry>
+      <origin xyz="0.046 0 -0.05334" rpy="3.14159265359 0 3.14159265359"/>
+    </collision>
+    <collision>
+      <geometry>
+        <mesh filename="package://ros2_descriptions/description/meshes/bravo7/1026 A.stl"/>
+      </geometry>
+      <origin xyz="0.046 0 -0.23534" rpy="3.14159265359 0 3.14159265359"/>
+    </collision>
+    <inertial>
+      <mass value="2.120"/>
+      <origin rpy="0 0 0" xyz="0.022 -0.004 -0.176"/>
+      <inertia
+        ixx="0.035166" ixy="0.0" ixz="0.0"
+        iyy="0.035981" iyz="0.0"
+        izz="0.003420"/>
     </inertial>
   </link>
@@ -132,5 +116,5 @@
     <axis xyz="0 -1 0"/>
     <limit effort="110.0" velocity="0.7854" lower="0.0" upper="3.2"/>
-    <dynamics damping="0.0" friction="0.08"/>
+    <dynamics damping="1430.0" friction="0.079"/>
   </joint>
   <link name="1026_0_joint_link">
@@ -150,21 +134,20 @@
     <collision>
       <geometry>
-        <cylinder radius="0.0408" length="0.02335"/>
-      </geometry>
-      <origin xyz="0 0.027275 0" rpy="1.57079632679 0 0"/>
-    </collision>
-    <collision>
-      <geometry>
-        <cylinder radius="0.0408" length="0.0946"/>
-      </geometry>
-      <origin xyz="0.0408 0 -0.0473" rpy="0 0 0"/>
-    </collision>
-    <inertial>
-      <mass value="1.000"/>
-      <origin rpy="0 0 0" xyz="0.0 0.0 0.25"/>
-      <inertia
-        ixx="0.015216803515624995" ixy="0.0" ixz="0.0"
-        iyy="0.015216803515624995" iyz="0.0"
-        izz="0.002095"/>
+        <mesh filename="package://ros2_descriptions/description/meshes/bravo7/1026 B.stl"/>
+      </geometry>
+    </collision>
+    <collision>
+      <geometry>
+        <mesh filename="package://ros2_descriptions/description/meshes/bravo7/1026 C.stl"/>
+      </geometry>
+      <origin xyz="0.0408 0 -0.0956" rpy="3.14159265359 0 0"/>
+    </collision>
+    <inertial>
+      <mass value="1.330"/>
+      <origin rpy="0 0 0" xyz="0.034 0.003 -0.046"/>
+      <inertia
+        ixx="0.001809" ixy="0.0" ixz="0.0"
+        iyy="0.002024" iyz="0.0"
+        izz="0.001557"/>
     </inertial>
   </link>
@@ -175,5 +158,5 @@
     <axis xyz="0 0 -1"/>
     <limit effort="110.0" velocity="0.7854"/>
-    <dynamics damping="0.0" friction="0.07"/>
+    <dynamics damping="1430.0" friction="0.079"/>
   </joint>
   <link name="1023_0_base_link">
@@ -187,21 +170,15 @@
     <collision>
       <geometry>
-        <cylinder radius="0.0408" length="0.059"/>
-      </geometry>
-      <origin xyz="0 0 0.0295" rpy="0 0 0"/>
-    </collision>
-    <collision>
-      <geometry>
-        <cylinder radius="0.0408" length="0.0599"/>
-      </geometry>
-      <origin xyz="0.0408 -0.01435 0.059" rpy="1.57079632679 0 0"/>
-    </collision>
-    <inertial>
-      <mass value="0.18790"/>
-      <origin rpy="0 0 0" xyz="0.0 0.0 0.0"/>
-      <inertia
-        ixx="8.062475833333332e-05" ixy="0.0" ixz="0.0"
-        iyy="8.062475833333332e-05" iyz="0.0"
-        izz="0.0001321171875"/>
+        <mesh filename="package://ros2_descriptions/description/meshes/bravo7/1023 A.stl"/>
+      </geometry>
+      <origin xyz="0 0 0.0054" rpy="0 0 3.14159265359"/>
+    </collision>
+    <inertial>
+      <mass value="1.330"/>
+      <origin rpy="0 0 0" xyz="0.028 -0.012 0.145"/>
+      <inertia
+        ixx="0.001983" ixy="0.0" ixz="0.0"
+        iyy="0.002676" iyz="0.0"
+        izz="0.001526"/>
     </inertial>
   </link>
@@ -212,5 +189,5 @@
     <axis xyz="0 -1 0"/>
     <limit effort="110.0" velocity="0.7854" lower="0.0" upper="3.2"/>
-    <dynamics damping="0.0" friction="0.07"/>
+    <dynamics damping="1430.0" friction="0.079"/>
   </joint>
   <link name="1023_0_joint_link">
@@ -230,21 +207,20 @@
     <collision>
       <geometry>
-        <cylinder radius="0.0408" length="0.02335"/>
-      </geometry>
-      <origin xyz="0 0.027275 0" rpy="1.57079632679 0 0"/>
-    </collision>
-    <collision>
-      <geometry>
-        <cylinder radius="0.0408" length="0.0946"/>
-      </geometry>
-      <origin xyz="0.0408 0 -0.0473" rpy="0 0 0"/>
-    </collision>
-    <inertial>
-      <mass value="0.18790"/>
-      <origin rpy="0 0 0" xyz="0.0 0.0 0.0"/>
-      <inertia
-        ixx="8.062475833333332e-05" ixy="0.0" ixz="0.0"
-        iyy="8.062475833333332e-05" iyz="0.0"
-        izz="0.0001321171875"/>
+        <mesh filename="package://ros2_descriptions/description/meshes/bravo7/1023 B.stl"/>
+      </geometry>
+    </collision>
+    <collision>
+      <geometry>
+        <mesh filename="package://ros2_descriptions/description/meshes/bravo7/1023 C.stl"/>
+      </geometry>
+      <origin xyz="0.0408 0 -0.0956" rpy="3.14159265359 0 3.14159265359"/>
+    </collision>
+    <inertial>
+      <mass value="0.970"/>
+      <origin rpy="0 0 0" xyz="0.031 0.006 -0.039"/>
+      <inertia
+        ixx="0.001272" ixy="0.0" ixz="0.0"
+        iyy="0.001511" iyz="0.0"
+        izz="0.001295"/>
     </inertial>
   </link>
@@ -255,5 +231,5 @@
     <axis xyz="0 0 -1"/>
     <limit effort="110.0" velocity="0.7854"/>
-    <dynamics damping="0.0" friction="0.07"/>
+    <dynamics damping="1430.0" friction="0.079"/>
   </joint>
   <link name="1038_base_link">
@@ -267,14 +243,15 @@
     <collision>
       <geometry>
-        <cylinder radius="0.0408" length="0.12535"/>
-      </geometry>
-    </collision>
-    <inertial>
-      <mass value="0.18790"/>
-      <origin rpy="0 0 0" xyz="0.0 0.0 0.0"/>
-      <inertia
-        ixx="8.062475833333332e-05" ixy="0.0" ixz="0.0"
-        iyy="8.062475833333332e-05" iyz="0.0"
-        izz="0.0001321171875"/>
+        <mesh filename="package://ros2_descriptions/description/meshes/bravo7/1038.stl"/>
+      </geometry>
+      <origin xyz="0 0 0.0054" rpy="0 0 0"/>
+    </collision>
+    <inertial>
+      <mass value="1.090"/>
+      <origin rpy="0 0 0" xyz="0.0 0.0 0.127"/>
+      <inertia
+        ixx="0.001977" ixy="0.0" ixz="0.0"
+        iyy="0.001986" iyz="0.0"
+        izz="0.001035"/>
     </inertial>
   </link>
