Commit message: finish jaws joints and links

File: description/bravo7.urdf.xacro (robot description, xacro)
@@ -28,4 +28,5 @@
   <!-- manipulator without jaws, for Pinocchio lib -->
   <xacro:include filename="$(find ros2_descriptions)/description/urdf/bravo7.description.urdf.xacro"/>
+  <!-- manipulator jaws -->
   <joint name="a_joint" type="prismatic">
     <!-- this parent link is the last link in bravo7.description -->
@@ -96,4 +97,36 @@
     </inertial>
   </link>
+  <joint name="rs2_301_joint" type="revolute">
+    <parent link="jaws_handle_link"/>
+    <child link="rs2_301_link"/>
+    <origin xyz="0.0241 -0.0268 0" rpy="3.14159265359 0 0"/>
+    <axis xyz="0 0 1"/>
+    <limit lower="0" upper="1.0" effort="10" velocity="10"/>
+    <mimic joint="rs2_300_joint" multiplier="1" offset="0"/>
+  </joint>
+  <link name="rs2_301_link">
+    <visual>
+      <geometry>
+        <mesh filename="package://ros2_descriptions/description/meshes/bravo7/RS2-301.stl"/>
+      </geometry>
+      <origin rpy="0 0 0" xyz="0.0 0.0 0.0"/>
+      <material name="bblack"/>
+    </visual>
+    <collision>
+      <geometry>
+        <mesh filename="package://ros2_descriptions/description/meshes/bravo7/RS2-301.stl"/>
+      </geometry>
+      <origin rpy="0 0 0" xyz="0.0 0.0 0.0"/>
+    </collision>
+    <inertial>
+      <mass value="0.10"/>
+      <origin rpy="0 0 0" xyz="0.0 0.0 0.0"/>
+      <inertia
+        ixx="0.000050" ixy="0.0" ixz="0.0"
+        iyy="0.000372" iyz="0.0"
+        izz="0.000376"/>
+    </inertial>
+  </link>
+  <!-- end of manipulator jaws -->
   <xacro:include filename="$(find ros2_descriptions)/description/ros2_control/bravo7.ros2_control.xacro"/>
   <xacro:bravo7_control/>

Commit message: Finish Bravo 7 model

File: description/bravo7.urdf.xacro (robot description, xacro)
@@ -53,15 +53,16 @@
     </visual>
     <collision>
+      <origin rpy="0 1.57079632679 0" xyz="0.015 0.0 0.0"/>
       <geometry>
-        <mesh filename="package://ros2_descriptions/description/meshes/bravo7/RS2-257.stl"/>
+        <cylinder radius="0.0356" length="0.030"/>
       </geometry>
     </collision>
     <inertial>
-      <mass value="0.44"/>
-      <origin rpy="0 0 0" xyz="0.0 0.0 0.0"/>
+      <mass value="0.512"/>
+      <origin rpy="0 0 0" xyz="0.004429 -0.000023 0"/>
       <inertia
-        ixx="0.000309" ixy="0.0" ixz="0.0"
-        iyy="0.002237" iyz="0.0"
-        izz="0.002258"/>
+        ixx="0.000379379" ixy="-5.1539957e-08" ixz="9.63256406e-08"
+        iyy="0.000275446" iyz="6.10616562e-08"
+        izz="0.000271025"/>
     </inertial>
   </link>
@@ -89,10 +90,10 @@
     </collision>
     <inertial>
-      <mass value="0.10"/>
-      <origin rpy="0 0 0" xyz="0.0 0.0 0.0"/>
+      <mass value="0.32667"/>
+      <origin rpy="0 0 0" xyz="0.050421 0.020670 0"/>
       <inertia
-        ixx="0.000050" ixy="0.0" ixz="0.0"
-        iyy="0.000372" iyz="0.0"
-        izz="0.000376"/>
+        ixx="7.1023328e-05" ixy="-0.0001197464" ixz="0.0"
+        iyy="0.000422552" iyz="0.0"
+        izz="0.000454988"/>
     </inertial>
   </link>
@@ -110,5 +111,4 @@
         <mesh filename="package://ros2_descriptions/description/meshes/bravo7/RS2-301.stl"/>
       </geometry>
-      <origin rpy="0 0 0" xyz="0.0 0.0 0.0"/>
       <material name="bblack"/>
     </visual>
@@ -117,13 +117,12 @@
         <mesh filename="package://ros2_descriptions/description/meshes/bravo7/RS2-301.stl"/>
       </geometry>
-      <origin rpy="0 0 0" xyz="0.0 0.0 0.0"/>
     </collision>
     <inertial>
-      <mass value="0.10"/>
-      <origin rpy="0 0 0" xyz="0.0 0.0 0.0"/>
+      <mass value="0.4555"/>
+      <origin rpy="0 0 0" xyz="0.052475 -0.022378 0"/>
       <inertia
-        ixx="0.000050" ixy="0.0" ixz="0.0"
-        iyy="0.000372" iyz="0.0"
-        izz="0.000376"/>
+        ixx="0.000151411" ixy="0.00015977" ixz="-1.318157e-09"
+        iyy="0.000574993" iyz="0.0"
+        izz="0.000570182"/>
     </inertial>
   </link>

File: description/urdf/bravo7.description.urdf.xacro (robot description, xacro)
@@ -38,10 +38,4 @@
       <material name="bblack"/>
     </visual>
-    <collision>
-      <geometry>
-        <mesh filename="package://ros2_descriptions/description/meshes/bravo7/1013 A.stl"/>
-      </geometry>
-      <origin rpy="0 0 3.14159265359" xyz="0 0 0"/>
-    </collision>
     <inertial>
       <mass value="1.620"/>
@@ -70,6 +64,7 @@
     <collision>
       <geometry>
-        <mesh filename="package://ros2_descriptions/description/meshes/bravo7/1013_merged.stl"/>
+        <cylinder radius="0.044" length="0.300"/>
       </geometry>
+      <origin rpy="0 0.041 0" xyz="0.044 0.0 -0.155"/>
     </collision>
     <inertial>
@@ -181,7 +176,7 @@
     <collision>
       <geometry>
-        <mesh filename="package://ros2_descriptions/description/meshes/bravo7/1038.stl"/>
+        <cylinder radius="0.040" length="0.120"/>
       </geometry>
-      <origin xyz="0 0 0.0054" rpy="0 0 0"/>
+      <origin rpy="0 0 0" xyz="0.0 0.0 0.0654"/>
     </collision>
     <inertial>

Commit message: Adjust URDF

File: description/bravo7.urdf.xacro (robot description, xacro)
@@ -1,6 +1,6 @@
 <?xml version="1.0"?>
 <robot xmlns:xacro="http://www.ros.org/wiki/xacro" name="Bravo7">
-  <material name="bblack">
-    <color rgba="0.3 0.3 0.3 1"/>
+  <material name="jaw_black">
+    <color rgba="0.401 0.403 0.403 1"/>
   </material>
   <link name="world">
@@ -39,5 +39,13 @@
   </joint>
   <!-- dummy frame for the prismatic joint -->
-  <link name="jaws_push_rod_link"/>
+  <link name="jaws_push_rod_link">
+    <inertial>
+      <mass value="0.09"/>
+      <inertia
+        ixx="0.000422552" ixy="0.0" ixz="0.0"
+        iyy="0.000422552" iyz="0.0"
+        izz="7.10233e-05"/>
+    </inertial>
+  </link>
   <joint name="jaws_base_joint" type="fixed">
     <parent link="jaws_base_link"/>
@@ -50,5 +58,5 @@
         <mesh filename="package://ros2_descriptions/description/meshes/bravo7/RS2-257.stl"/>
       </geometry>
-      <material name="bblack"/>
+      <material name="jaw_black"/>
     </visual>
     <collision>
@@ -81,5 +89,5 @@
       </geometry>
       <origin rpy="3.14159265359 0 0" xyz="0.0 0.0 0.0"/>
-      <material name="bblack"/>
+      <material name="jaw_black"/>
     </visual>
     <collision>
@@ -111,5 +119,5 @@
         <mesh filename="package://ros2_descriptions/description/meshes/bravo7/RS2-301.stl"/>
       </geometry>
-      <material name="bblack"/>
+      <material name="jaw_black"/>
     </visual>
     <collision>

File: description/urdf/bravo7.description.urdf.xacro (robot description, xacro)
@@ -1,4 +1,7 @@
 <?xml version="1.0" encoding="utf-8"?>
 <robot xmlns:xacro="http://wiki.ros.org/xacro" name="Bravo7">
+  <material name="bblack">
+    <color rgba="0.3 0.3 0.3 1"/>
+  </material>
   <link name="base_link">
     <visual>
@@ -22,10 +25,10 @@
     </inertial>
   </link>
-  <joint name="g_joint" type="continuous">
+  <joint name="g_joint" type="revolute">
     <parent link="base_link"/>
     <child link="1013_base_link"/>
     <origin xyz="0.0665 0 0.0858" rpy="0 0 3.14159265359"/>
     <axis xyz="0 0 -1"/>
-    <limit effort="110.0" velocity="0.7854"/>
+    <limit effort="110.0" velocity="0.7854" lower="-6.28318530718" upper="6.28318530718"/>
     <dynamics damping="1430.0" friction="0.079"/>
   </joint>
@@ -102,10 +105,10 @@
     </inertial>
   </link>
-  <joint name="d_joint" type="continuous">
+  <joint name="d_joint" type="revolute">
     <parent link="1026_0_joint_link"/>
     <child link="1023_0_base_link"/>
     <origin xyz="0.0408 0 -0.0956" rpy="3.14159265359 0 0"/>
     <axis xyz="0 0 -1"/>
-    <limit effort="110.0" velocity="0.7854"/>
+    <limit effort="110.0" velocity="0.7854" lower="-6.28318530718" upper="6.28318530718"/>
     <dynamics damping="1430.0" friction="0.079"/>
   </joint>
@@ -158,10 +161,10 @@
     </inertial>
   </link>
-  <joint name="b_joint" type="continuous">
+  <joint name="b_joint" type="revolute">
     <parent link="1023_0_joint_link"/>
     <child link="1038_base_link"/>
     <origin xyz="0.0408 0 -0.0956" rpy="3.14159265359 0 3.14159265359"/>
     <axis xyz="0 0 -1"/>
-    <limit effort="110.0" velocity="0.7854"/>
+    <limit effort="110.0" velocity="0.7854" lower="-6.28318530718" upper="6.28318530718"/>
     <dynamics damping="1430.0" friction="0.079"/>
   </joint>

Commit message: Adjustment to use Bravo 7 with bullet-featherstone

File: description/bravo7.urdf.xacro (robot description, xacro)
@@ -36,5 +36,5 @@
     <axis xyz="1 0 0"/>
     <limit lower="0.000" upper="0.010" effort="10" velocity="10"/>
-    <dynamics damping="0.14833" friction="13.166"/>
+    <dynamics damping="0.074" friction="0.07"/>
   </joint>
   <!-- dummy frame for the prismatic joint -->
@@ -45,5 +45,5 @@
         ixx="0.000422552" ixy="0.0" ixz="0.0"
         iyy="0.000422552" iyz="0.0"
-        izz="7.10233e-05"/>
+        izz="1.10233e-04"/>
     </inertial>
   </link>
@@ -70,6 +70,6 @@
       <origin rpy="0 0 0" xyz="0.004429 -0.000023 0"/>
       <inertia
-        ixx="0.000379379" ixy="-5.1539957e-08" ixz="9.63256406e-08"
-        iyy="0.000275446" iyz="6.10616562e-08"
+        ixx="0.000379379" ixy="0.0" ixz="0.0"
+        iyy="0.000275446" iyz="0.0"
         izz="0.000271025"/>
     </inertial>
@@ -101,5 +101,5 @@
       <origin rpy="0 0 0" xyz="0.050421 0.020670 0"/>
       <inertia
-        ixx="7.1023328e-05" ixy="-0.0001197464" ixz="0.0"
+        ixx="1.00232e-04" ixy="0.0" ixz="0.0"
         iyy="0.000422552" iyz="0.0"
         izz="0.000454988"/>
@@ -130,5 +130,5 @@
       <origin rpy="0 0 0" xyz="0.052475 -0.022378 0"/>
       <inertia
-        ixx="0.000151411" ixy="0.00015977" ixz="-1.318157e-09"
+        ixx="0.000151411" ixy="0.0" ixz="0.0"
         iyy="0.000574993" iyz="0.0"
         izz="0.000570182"/>

File: description/ros2_control/bravo7.ros2_control.xacro (robot description, xacro)
@@ -18,5 +18,7 @@
           <param name="initial_value">${config['initial']['g_joint']}</param>
         </state_interface>
-        <state_interface name="velocity"/>
+        <state_interface name="velocity">
+          <param name="initial_value">0.0</param>
+        </state_interface>
         <state_interface name="effort"/>
       </joint>
@@ -26,5 +28,7 @@
           <param name="initial_value">${config['initial']['f_joint']}</param>
         </state_interface>
-        <state_interface name="velocity"/>
+        <state_interface name="velocity">
+          <param name="initial_value">0.0</param>
+        </state_interface>
         <state_interface name="effort"/>
       </joint>
@@ -34,5 +38,7 @@
           <param name="initial_value">${config['initial']['e_joint']}</param>
         </state_interface>
-        <state_interface name="velocity"/>
+        <state_interface name="velocity">
+          <param name="initial_value">0.0</param>
+        </state_interface>
         <state_interface name="effort"/>
       </joint>
@@ -42,5 +48,7 @@
           <param name="initial_value">${config['initial']['d_joint']}</param>
         </state_interface>
-        <state_interface name="velocity"/>
+        <state_interface name="velocity">
+          <param name="initial_value">0.0</param>
+        </state_interface>
         <state_interface name="effort"/>
       </joint>
@@ -50,5 +58,7 @@
           <param name="initial_value">${config['initial']['c_joint']}</param>
         </state_interface>
-        <state_interface name="velocity"/>
+        <state_interface name="velocity">
+          <param name="initial_value">0.0</param>
+        </state_interface>
         <state_interface name="effort"/>
       </joint>
@@ -58,5 +68,7 @@
           <param name="initial_value">${config['initial']['b_joint']}</param>
         </state_interface>
-        <state_interface name="velocity"/>
+        <state_interface name="velocity">
+          <param name="initial_value">0.0</param>
+        </state_interface>
         <state_interface name="effort"/>
       </joint>
@@ -66,5 +78,7 @@
           <param name="initial_value">${config['initial']['a_joint']}</param>
         </state_interface>
-        <state_interface name="velocity"/>
+        <state_interface name="velocity">
+          <param name="initial_value">0.0</param>
+        </state_interface>
         <state_interface name="effort"/>
       </joint>

File: description/urdf/bravo7.description.urdf.xacro (robot description, xacro)
@@ -31,5 +31,5 @@
     <axis xyz="0 0 -1"/>
     <limit effort="110.0" velocity="0.7854" lower="-6.28318530718" upper="6.28318530718"/>
-    <dynamics damping="1430.0" friction="0.079"/>
+    <dynamics damping="7.15" friction="0.079"/>
   </joint>
   <link name="1013_base_link">
@@ -41,4 +41,10 @@
       <material name="bblack"/>
     </visual>
+    <collision>
+      <geometry>
+        <mesh filename="package://ros2_descriptions/description/meshes/bravo7/1013 A.stl"/>
+      </geometry>
+      <origin rpy="0 0 3.14159265359" xyz="0 0 0"/>
+    </collision>
     <inertial>
       <mass value="1.620"/>
@@ -56,5 +62,5 @@
     <axis xyz="0 -1 0"/>
     <limit effort="110.0" velocity="0.7854" lower="0.0" upper="3.2"/>
-    <dynamics damping="1430.0" friction="0.079"/>
+    <dynamics damping="8.90" friction="0.079"/>
   </joint>
   <link name="1013_joint_link">
@@ -86,5 +92,5 @@
     <axis xyz="0 -1 0"/>
     <limit effort="110.0" velocity="0.7854" lower="0.0" upper="3.2"/>
-    <dynamics damping="1430.0" friction="0.079"/>
+    <dynamics damping="7.1" friction="0.079"/>
   </joint>
   <link name="1026_0_joint_link">
@@ -96,4 +102,10 @@
       <material name="bblack"/>
     </visual>
+    <collision>
+      <geometry>
+        <mesh filename="package://ros2_descriptions/description/meshes/bravo7/1026.stl"/>
+      </geometry>
+      <origin xyz="-0.0052 0 0"/>
+    </collision>
     <inertial>
       <mass value="1.330"/>
@@ -111,5 +123,5 @@
     <axis xyz="0 0 -1"/>
     <limit effort="110.0" velocity="0.7854" lower="-6.28318530718" upper="6.28318530718"/>
-    <dynamics damping="1430.0" friction="0.079"/>
+    <dynamics damping="5.1" friction="0.079"/>
   </joint>
   <link name="1023_0_base_link">
@@ -142,5 +154,5 @@
     <axis xyz="0 -1 0"/>
     <limit effort="110.0" velocity="0.7854" lower="0.0" upper="3.2"/>
-    <dynamics damping="1430.0" friction="0.079"/>
+    <dynamics damping="6.59" friction="0.079"/>
   </joint>
   <link name="1023_0_joint_link">
@@ -152,4 +164,10 @@
       <material name="bblack"/>
     </visual>
+    <collision>
+      <geometry>
+        <mesh filename="package://ros2_descriptions/description/meshes/bravo7/1026.stl"/>
+      </geometry>
+      <origin xyz="-0.0052 0.001 0"/>
+    </collision>
     <inertial>
       <mass value="0.970"/>
@@ -167,5 +185,5 @@
     <axis xyz="0 0 -1"/>
     <limit effort="110.0" velocity="0.7854" lower="-6.28318530718" upper="6.28318530718"/>
-    <dynamics damping="1430.0" friction="0.079"/>
+    <dynamics damping="1.57" friction="0.079"/>
   </joint>
   <link name="1038_base_link">

Commit message: Deprecate bullet-featherstone

File: description/bravo7.urdf.xacro (robot description, xacro)
@@ -26,19 +26,15 @@
     <origin xyz="-0.045 0 0.60" rpy="0 0 0"/>
   </joint>
-  <!--
-    URDF joint dynamics and link inertia were adjusted for a stable
-    execution with 'gz-physics-bullet-featherstone-plugin'.
-  -->
   <!-- manipulator without jaws, for Pinocchio lib -->
   <xacro:include filename="$(find ros2_descriptions)/description/urdf/bravo7.description.urdf.xacro"/>
   <!-- manipulator jaws -->
   <joint name="a_joint" type="prismatic">
-    <!-- this parent link is the last link in bravo7.description -->
+    <!-- This parent is the last link in bravo7.description -->
     <parent link="jaws_base_link"/>
     <child link="jaws_push_rod_link"/>
     <origin rpy="0 0 0" xyz="0.009 0 0"/>
     <axis xyz="1 0 0"/>
-    <limit lower="0.000" upper="0.010" effort="10" velocity="10"/>
-    <dynamics damping="0.074" friction="0.07"/>
+    <limit lower="0.000" upper="0.010" effort="800" velocity="0.025"/>
+    <dynamics damping="0.074" friction="0.079"/>
   </joint>
   <!-- dummy frame for the prismatic joint -->
@@ -84,6 +80,7 @@
     <origin xyz="0.0241 0.0268 0" rpy="0 0 0"/>
     <axis xyz="0 0 1"/>
-    <limit lower="0" upper="1.0" effort="10" velocity="10"/>
-    <mimic joint="a_joint" multiplier="54" offset="0"/>
+    <limit lower="-0.005" upper="1.005" effort="400" velocity="0.7854"/>
+    <!-- Mimic is not supported by Dart -->
+    <!--mimic joint="a_joint" multiplier="54" offset="0"/-->
   </joint>
   <link name="rs2_300_link">
@@ -115,6 +112,6 @@
     <origin xyz="0.0241 -0.0268 0" rpy="3.14159265359 0 0"/>
     <axis xyz="0 0 1"/>
-    <limit lower="0" upper="1.0" effort="10" velocity="10"/>
-    <mimic joint="rs2_300_joint" multiplier="1" offset="0"/>
+    <limit lower="-0.005" upper="1.005" effort="400" velocity="0.7854"/>
+    <!--mimic joint="rs2_300_joint" multiplier="1" offset="0"/-->
   </joint>
   <link name="rs2_301_link">

File: description/ros2_control/bravo7.ros2_control.xacro (robot description, xacro)
@@ -74,7 +74,27 @@
       </joint>
       <joint name="a_joint">
-        <command_interface name="effort"/>
+        <command_interface name="position"/>
         <state_interface name="position">
           <param name="initial_value">${config['initial']['a_joint']}</param>
+        </state_interface>
+        <state_interface name="velocity">
+          <param name="initial_value">0.0</param>
+        </state_interface>
+        <state_interface name="effort"/>
+      </joint>
+      <joint name="rs2_300_joint">
+        <command_interface name="position"/>
+        <state_interface name="position">
+          <param name="initial_value">0.02</param>
+        </state_interface>
+        <state_interface name="velocity">
+          <param name="initial_value">0.0</param>
+        </state_interface>
+        <state_interface name="effort"/>
+      </joint>
+      <joint name="rs2_301_joint">
+        <command_interface name="position"/>
+        <state_interface name="position">
+          <param name="initial_value">0.02</param>
         </state_interface>
         <state_interface name="velocity">

File: description/urdf/bravo7.description.urdf.xacro (robot description, xacro)
@@ -31,5 +31,5 @@
     <axis xyz="0 0 -1"/>
     <limit effort="110.0" velocity="0.7854" lower="-6.28318530718" upper="6.28318530718"/>
-    <dynamics damping="7.15" friction="0.079"/>
+    <dynamics damping="7.22" friction="0.079"/>
   </joint>
   <link name="1013_base_link">
@@ -62,5 +62,5 @@
     <axis xyz="0 -1 0"/>
     <limit effort="110.0" velocity="0.7854" lower="0.0" upper="3.2"/>
-    <dynamics damping="8.90" friction="0.079"/>
+    <dynamics damping="13.90" friction="0.079"/>
   </joint>
   <link name="1013_joint_link">
@@ -92,5 +92,5 @@
     <axis xyz="0 -1 0"/>
     <limit effort="110.0" velocity="0.7854" lower="0.0" upper="3.2"/>
-    <dynamics damping="7.1" friction="0.079"/>
+    <dynamics damping="10.18" friction="0.079"/>
   </joint>
   <link name="1026_0_joint_link">
@@ -123,5 +123,5 @@
     <axis xyz="0 0 -1"/>
     <limit effort="110.0" velocity="0.7854" lower="-6.28318530718" upper="6.28318530718"/>
-    <dynamics damping="5.1" friction="0.079"/>
+    <dynamics damping="7.13" friction="0.079"/>
   </joint>
   <link name="1023_0_base_link">
@@ -154,5 +154,5 @@
     <axis xyz="0 -1 0"/>
     <limit effort="110.0" velocity="0.7854" lower="0.0" upper="3.2"/>
-    <dynamics damping="6.59" friction="0.079"/>
+    <dynamics damping="9.59" friction="0.079"/>
   </joint>
   <link name="1023_0_joint_link">
@@ -184,6 +184,6 @@
     <origin xyz="0.0408 0 -0.0956" rpy="3.14159265359 0 3.14159265359"/>
     <axis xyz="0 0 -1"/>
-    <limit effort="110.0" velocity="0.7854" lower="-6.28318530718" upper="6.28318530718"/>
-    <dynamics damping="1.57" friction="0.079"/>
+    <limit effort="20.0" velocity="0.7854" lower="-6.28318530718" upper="6.28318530718"/>
+    <dynamics damping="3.78" friction="0.079"/>
   </joint>
   <link name="1038_base_link">
@@ -197,7 +197,7 @@
     <collision>
       <geometry>
-        <cylinder radius="0.040" length="0.120"/>
-      </geometry>
-      <origin rpy="0 0 0" xyz="0.0 0.0 0.0654"/>
+        <mesh filename="package://ros2_descriptions/description/meshes/bravo7/1038.stl"/>
+      </geometry>
+      <origin xyz="0 0 0.0054" rpy="0 0 0"/>
     </collision>
     <inertial>
