Commit message: Refact HyL setup argument

File: description/hyl.urdf.xacro (robot description, xacro)
@@ -1,5 +1,6 @@
 <?xml version="1.0" ?>
 <robot xmlns:xacro="http://www.ros.org/wiki/xacro" name="HyL">
-  <xacro:arg name="fixed" default="false"/>
+  <xacro:arg name="setup" default=""/>
+  <xacro:property name="bench_setup" value="$(arg setup)"/>
   <material name="StaticBlue">
     <color rgba="0.20 1.0 1.0 0.9"/>
@@ -14,5 +15,5 @@
     </visual>
   </link>
-  <xacro:if value="$(arg fixed)">
+  <xacro:if value="${bench_setup == 'fixed'}">
     <joint name="support_joint" type="fixed">
       <origin xyz="0.0 0.04 0.7" rpy="0 0 0" />
@@ -21,5 +22,5 @@
     </joint>
   </xacro:if>
-  <xacro:unless value="$(arg fixed)">
+  <xacro:unless value="${bench_setup == 'fixed'}">
     <joint name="support_joint" type="prismatic">
       <origin xyz="0.0 0.04 0.5" rpy="0 0 0" />
@@ -33,4 +34,4 @@
   <xacro:include filename="$(find ros2_descriptions)/description/urdf/hyl.description.urdf.xacro" />
   <xacro:include filename="$(find ros2_descriptions)/description/ros2_control/hyl.ros2_control.xacro" />
-  <xacro:hyq_control fixed_support="$(arg fixed)"/>
+  <xacro:hyl_control fixed_support="${bench_setup == 'fixed'}"/>
 </robot>

File: description/ros2_control/hyl.ros2_control.xacro (robot description, xacro)
@@ -1,5 +1,5 @@
 <?xml version="1.0"?>
 <robot xmlns:xacro="http://www.ros.org/wiki/xacro">
-  <xacro:macro name="hyq_control" params="fixed_support">
+  <xacro:macro name="hyl_control" params="fixed_support">
     <xacro:property name="robot_yaml" value="$(find ros2_descriptions)/config/hyl.yaml"/>
     <xacro:property name="config" value="${xacro.load_yaml(robot_yaml)}"/>
